File: ESR_NM8032.sch (EAGLE design)
At the start: 65 parts, among them J1 J5MM

Commit message: 2
Parts:
- 3C10, 3C7: device rcl:C-EU025-025X050 -> rcl:C-EUC0805
- 3C6: device rc-elektronik:C-EU025-024X044 -> rc-elektronik:C-EUC0805
- C2: device rcl:C-EUC0805 -> rcl:C-EU050-025X075
- C9: device rcl:CPOL-EUE2.5-5 -> rcl:CPOL-EUE15-5AXIAL
- R1: device rcl:R-EU_M0805 -> rcl:R-EU_0207/10
Changed lines of the file:
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@@
 <setting verticaltext="up"/>
 </settings>
-<grid distance="100" unitdist="mil" unit="mil" style="lines" multiple="1" display="yes" altdistance="0.01" altunitdist="inch" altunit="inch"/>
+<grid distance="0.1" unitdist="inch" unit="mil" style="lines" multiple="1" display="yes" altdistance="0.01" altunitdist="inch" altunit="inch"/>
 <layers>
 <layer number="1" name="Top" color="4" fill="1" visible="yes" active="no"/>
@@
 <part name="DD1" library="40xx" deviceset="4049" device="D"/>
 <part name="C1" library="rcl" deviceset="C-EU" device="C0805" value="330"/>
-<part name="R1" library="rcl" deviceset="R-EU_" device="M0805" value="20k"/>
-<part name="C2" library="rcl" deviceset="C-EU" device="C0805" value="220n"/>
+<part name="R1" library="rcl" deviceset="R-EU_" device="0207/10" value="20k"/>
+<part name="C2" library="rcl" deviceset="C-EU" device="050-025X075" value="220n"/>
 <part name="LED1" library="led" deviceset="LED" device="SML0603"/>
 <part name="LED2" library="led" deviceset="LED" device="SML0603"/>
@@
 <part name="R8" library="rcl" deviceset="R-EU_" device="R1206W" value="5k6"/>
 <part name="GND4" library="supply1" deviceset="GND" device=""/>
-<part name="3C6" library="rc-elektronik" deviceset="C-EU" device="025-024X044" value="100n"/>
+<part name="3C6" library="rc-elektronik" deviceset="C-EU" device="C0805" value="100n"/>
 <part name="DA4" library="mc34063" deviceset="MC34063" device="AD"/>
 <part name="3R5" library="rcl" deviceset="R-EU_" device="0204/7" value="220"/>
@@
 <part name="3L2" library="rcl" deviceset="L-US" device="0207/10" value="100uh"/>
 <part name="3VD2" library="diode" deviceset="SCHOTTKY-DIODE" device="SMD" value="SS12"/>
-<part name="3C7" library="rcl" deviceset="C-EU" device="025-025X050" value="1n"/>
+<part name="3C7" library="rcl" deviceset="C-EU" device="C0805" value="1n"/>
 <part name="GND7" library="supply1" deviceset="GND" device=""/>
 <part name="GND8" library="supply1" deviceset="GND" device=""/>
@@
 <part name="3C8" library="HWProgUSB" deviceset="RCL_CPOL-EU" device="E3.5-8" value="470µ / 10V"/>
 <part name="3C9" library="HWProgUSB" deviceset="RCL_CPOL-EU" device="E3.5-8" value="100µ 16V"/>
-<part name="3C10" library="rcl" deviceset="C-EU" device="025-025X050" value="100n"/>
+<part name="3C10" library="rcl" deviceset="C-EU" device="C0805" value="100n"/>
 <part name="R9" library="rcl" deviceset="R-EU_" device="R0805" value="10k"/>
 <part name="GND5" library="supply1" deviceset="GND" device=""/>
@@
 <part name="JP4" library="pinhead" deviceset="PINHD-1X2" device=""/>
 <part name="3L1" library="rcl" deviceset="L-US" device="0207/10" value="100uh"/>
-<part name="C9" library="rcl" deviceset="CPOL-EU" device="E2.5-5" value="470x6v3"/>
+<part name="C9" library="rcl" deviceset="CPOL-EU" device="E15-5AXIAL" value="470x6v3"/>
 <part name="C10" library="rcl" deviceset="C-EU" device="C0805" value="330n"/>
 <part name="3L3" library="rcl" deviceset="L-US" device="0207/10" value="100uh"/>

Commit message: 3
Parts:
- added 3C1: 100n, rcl:C-EUC0805
- added 3C2: 100µ 16V, HWProgUSB:RCL_CPOL-EUE3.5-8
- 3R5: value 220 -> 180; device rcl:R-EU_0204/7 -> rcl:R-EU_M0805
- 3R6: device rcl:R-EU_0204/7 -> rcl:R-EU_M1206
- 3R7: value 20k -> 9k1
- 3R8: value 2k2 -> 2k4
- C8: device rcl:C-EUC0805 -> rcl:C-EU050-025X075
- R8: device rcl:R-EU_R1206W -> rcl:R-EU_0207/10
Connections:
- net GND: now also 3C1.1, 3C2.-
- net V+: now also 3C1.2, 3C2.+
Changed lines of the file:
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@@
 <part name="C6" library="rcl" deviceset="C-EU" device="C0805" value="220n"/>
 <part name="C5" library="rcl" deviceset="C-EU" device="C0805" value="220n"/>
-<part name="R8" library="rcl" deviceset="R-EU_" device="R1206W" value="5k6"/>
+<part name="R8" library="rcl" deviceset="R-EU_" device="0207/10" value="5k6"/>
 <part name="GND4" library="supply1" deviceset="GND" device=""/>
 <part name="3C6" library="rc-elektronik" deviceset="C-EU" device="C0805" value="100n"/>
 <part name="DA4" library="mc34063" deviceset="MC34063" device="AD"/>
-<part name="3R5" library="rcl" deviceset="R-EU_" device="0204/7" value="220"/>
-<part name="3R6" library="rcl" deviceset="R-EU_" device="0204/7" value="0.5-1"/>
+<part name="3R5" library="rcl" deviceset="R-EU_" device="M0805" value="180"/>
+<part name="3R6" library="rcl" deviceset="R-EU_" device="M1206" value="0.5-1"/>
 <part name="GND6" library="supply1" deviceset="GND" device=""/>
-<part name="3R7" library="rcl" deviceset="R-EU_" device="M0805" value="20k"/>
-<part name="3R8" library="rcl" deviceset="R-EU_" device="M0805" value="2k2"/>
+<part name="3R7" library="rcl" deviceset="R-EU_" device="M0805" value="9k1"/>
+<part name="3R8" library="rcl" deviceset="R-EU_" device="M0805" value="2k4"/>
 <part name="3L2" library="rcl" deviceset="L-US" device="0207/10" value="100uh"/>
 <part name="3VD2" library="diode" deviceset="SCHOTTKY-DIODE" device="SMD" value="SS12"/>
@@
 <part name="C7" library="rcl" deviceset="CPOL-EU" device="E2.5-5" value="10m"/>
 <part name="R10" library="rcl" deviceset="R-EU_" device="R0805" value="10k"/>
-<part name="C8" library="rcl" deviceset="C-EU" device="C0805" value="220n"/>
+<part name="C8" library="rcl" deviceset="C-EU" device="050-025X075" value="220n"/>
 <part name="R11" library="rcl" deviceset="R-EU_" device="R0805" value="10k"/>
 <part name="R12" library="rcl" deviceset="R-EU_" device="R0805" value="10k"/>
@@
 <part name="DA2" library="ESR_NM8032" deviceset="K157DA1" device=""/>
 <part name="P+4" library="supply1" deviceset="V+" device=""/>
+<part name="3C1" library="rcl" deviceset="C-EU" device="C0805" value="100n"/>
+<part name="GND1" library="supply1" deviceset="GND" device=""/>
+<part name="3C2" library="HWProgUSB" deviceset="RCL_CPOL-EU" device="E3.5-8" value="100µ 16V"/>
+<part name="GND2" library="supply1" deviceset="GND" device=""/>
 </parts>
 <sheets>
@@
 <attribute name="VALUE" x="223.52" y="185.42" size="1.778" layer="96" rot="R180"/>
 </instance>
+<instance part="3C1" gate="G$1" x="119.38" y="40.64" smashed="yes" rot="R180">
+<attribute name="NAME" x="123.444" y="41.021" size="1.778" layer="95"/>
+<attribute name="VALUE" x="122.174" y="38.481" size="1.778" layer="96"/>
+</instance>
+<instance part="GND1" gate="1" x="119.38" y="33.02"/>
+<instance part="3C2" gate="G$1" x="109.22" y="43.18"/>
+<instance part="GND2" gate="1" x="109.22" y="33.02"/>
 </instances>
 <busses>
@@
 <wire x1="76.2" y1="116.84" x2="76.2" y2="111.76" width="0.1524" layer="91"/>
 <pinref part="GND4" gate="1" pin="GND"/>
+</segment>
+<segment>
+<pinref part="3C1" gate="G$1" pin="1"/>
+<pinref part="GND1" gate="1" pin="GND"/>
+<wire x1="119.38" y1="38.1" x2="119.38" y2="35.56" width="0.1524" layer="91"/>
+</segment>
+<segment>
+<pinref part="GND2" gate="1" pin="GND"/>
+<pinref part="3C2" gate="G$1" pin="-"/>
+<wire x1="109.22" y1="35.56" x2="109.22" y2="38.1" width="0.1524" layer="91"/>
 </segment>
 </net>
@@
 <pinref part="P+1" gate="1" pin="V+"/>
 <wire x1="119.38" y1="68.58" x2="119.38" y2="71.12" width="0.1524" layer="91"/>
-</segment>
-</net>
+<pinref part="3C1" gate="G$1" pin="2"/>
+<wire x1="119.38" y1="45.72" x2="119.38" y2="53.34" width="0.1524" layer="91"/>
+<junction x="119.38" y="68.58"/>
+<pinref part="3C2" gate="G$1" pin="+"/>
+<wire x1="119.38" y1="53.34" x2="119.38" y2="68.58" width="0.1524" layer="91"/>
+<wire x1="109.22" y1="45.72" x2="109.22" y2="53.34" width="0.1524" layer="91"/>
+<wire x1="109.22" y1="53.34" x2="119.38" y2="53.34" width="0.1524" layer="91"/>
+<junction x="119.38" y="53.34"/>
+</segment>
+</net>

Commit message: 4
Parts:
- removed J1: J5MM, jumper:J5MM
- added C11: 470x6v3, rcl:CPOL-EUE15-5AXIAL
- added JP1: (no value), pinhead:PINHD-1X2
- 3R7: device rcl:R-EU_M0805 -> rcl:R-EU_0207/12
- C8: device rcl:C-EU050-025X075 -> rcl:C-EU075-032X103
Connections:
- removed net N$22: DA3.MODE, J1.1
- net +5V: now also JP1.1
- net GND: now also JP1.2
- net V+: now also DA3.MODE; no longer J1.2
Other:
- moved on the sheet: C10, C3, C4, C5, C7, C8, DA3, LED11, LED12, LED13, LED14, LED15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

Commit message: .
Parts:
- removed LED1, LED10, LED2, LED3, LED4, LED5, LED6, LED7, LED8, LED9: (no value), led:LEDSML0603
- removed LED11, LED12, LED13, LED14, LED15, LED16, LED17, LED18, LED19, LED20: (no value), led:LED3MM
- added HL1, HL10, HL2, HL3, HL4, HL5, HL6, HL7, HL8, HL9: (no value), led:LED3MM
Connections:
- removed net N$28: LED1.A, LED10.A, LED2.A, LED3.A, LED4.A, LED5.A, LED6.A, LED7.A, LED8.A, LED9.A
- net N$10: now also HL6.C; no longer LED16.C
- net N$11: now also HL7.C; no longer LED17.C
- net N$12: now also HL8.C; no longer LED18.C
- net N$13: now also HL9.C; no longer LED19.C
- net N$14: now also HL10.C; no longer LED20.C
- net N$3: now also HL1.C; no longer LED11.C
- net N$5: now also HL2.C; no longer LED12.C
- net N$7: now also HL3.C; no longer LED13.C
- net N$8: now also HL4.C; no longer LED14.C
- net N$9: now also HL5.C; no longer LED15.C
- net V+: now also HL1.A, HL10.A, HL2.A, HL3.A, HL4.A, HL5.A, HL6.A, HL7.A, HL8.A, HL9.A; no longer LED11.A, LED12.A, LED13.A, LED14.A, LED15.A, LED16.A, LED17.A, LED18.A, LED19.A, LED20.A
Other:
- moved on the sheet: 3C1, 3C10, 3C2, 3C6, 3C7, 3C8, 3C9, 3L1, 3L2, 3L3, 3R5, 3R6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

Commit message: 5
Parts:
- removed 3C2: 100µ 16V, HWProgUSB:RCL_CPOL-EUE3.5-8
- C11: value 470x6v3 -> 330n; device rcl:CPOL-EUE15-5AXIAL -> rcl:C-EUC0805
- C3: value 330n -> 220n
- C5: value 220n -> 10m; device rcl:C-EUC0805 -> rcl:CPOL-EUE2.5-5
- C6: device rcl:C-EUC0805 -> rcl:C-EU075-032X103
- C7: value 10m -> 220n; device rcl:CPOL-EUE2.5-5 -> rcl:C-EUC0805
- C8: value 220n -> 100µ 16V; device rcl:C-EU075-032X103 -> HWProgUSB:RCL_CPOL-EUE3.5-8
- R10: value 10k -> 4k7
- R11: value 10k -> 1k2
- R12: value 10k -> 3k
- R2: value 1k2 -> 2k; device rcl:R-EU_R0805 -> rcl:R-EU_M0805
- R3: value 4k7 -> 110; device rcl:R-EU_R0805 -> rcl:R-EU_M0805
- R4: value 3k -> 10k
- R5: value 30k -> 5k6; device rcl:R-EU_R0805 -> rcl:R-EU_0207/10
- R6: value 2k -> 10k; device rcl:R-EU_M0805 -> rcl:R-EU_R0805
- R7: value 110 -> 10k; device rcl:R-EU_M0805 -> rcl:R-EU_R0805
- R8: value 5k6 -> 10k; device rcl:R-EU_0207/10 -> rcl:R-EU_R0805
- R9: value 10k -> 30k
- renumbered 3C1 to C17, 3C10 to C15, 3C6 to C12, 3C7 to C16, 3C8 to C13, 3C9 to C14, 3L1 to L1, 3L2 to L2, 3L3 to L3, 3R5 to R14, 3R6 to R13, 3R7 to R16, 3R8 to R15, JP1 to X3, JP2 to SW1, JP3 to X1, JP4 to X2
Connections:
- removed net N$27: C5.2, X2.2
- new net N$22: C4.2, R5.1
- net GND: now also C11.2, C5.-, C7.2, C8.-, R10.1, R11.1, R8.1; no longer 3C2.-, C3.2, C4.2, C7.-, R2.1, R3.1, R5.1
- net N$19: now also C4.1, X2.2; no longer C5.1, R8.1
- net N$2: now also C3.1; no longer C6.1
- net N$20: now also R11.2; no longer R2.2
- net N$21: now also R10.2, R12.1; no longer R3.2, R4.1
- net N$23: now also R3.1; no longer R7.1
- net N$24: now also C7.1, R9.2; no longer C4.1, R5.2
- net N$25: now also R2.1; no longer R6.1
- net N$26: now also C3.2, R2.2, R3.2; no longer C6.2, R6.2, R7.2
- net N$29: now also R5.2, R6.1; no longer R11.1, R8.2
- net N$35: now also C6.1, R7.2; no longer C8.1, R10.2
- net N$36: now also C6.2, R6.2; no longer C8.2, R11.2
- net N$37: now also C5.+, R4.1, R7.1, R8.2; no longer C7.+, R10.1, R12.1, R9.2
- net V+: now also C11.1, C8.+; no longer 3C2.+, C3.1
Other:
- moved on the sheet: C3, C4, C6, R10, R11, R12, R2, R3, R4, R5, R6, R7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

Commit message: 6
Parts:
- added C18: 100µ 16V, HWProgUSB:RCL_CPOL-EUE2-5
Connections:
- net GND: now also C18.-
- net V+: now also C18.+
Changed lines of the file:
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@@
 <grid distance="0.1" unitdist="inch" unit="mil" style="lines" multiple="1" display="yes" altdistance="0.01" altunitdist="inch" altunit="inch"/>
 <layers>
-<layer number="1" name="Top" color="4" fill="1" visible="no" active="no"/>
-<layer number="2" name="Route2" color="1" fill="3" visible="no" active="no"/>
-<layer number="3" name="Route3" color="4" fill="3" visible="no" active="no"/>
-<layer number="4" name="Route4" color="1" fill="4" visible="no" active="no"/>
-<layer number="5" name="Route5" color="4" fill="4" visible="no" active="no"/>
-<layer number="6" name="Route6" color="1" fill="8" visible="no" active="no"/>
-<layer number="7" name="Route7" color="4" fill="8" visible="no" active="no"/>
-<layer number="8" name="Route8" color="1" fill="2" visible="no" active="no"/>
-<layer number="9" name="Route9" color="4" fill="2" visible="no" active="no"/>
-<layer number="10" name="Route10" color="1" fill="7" visible="no" active="no"/>
-<layer number="11" name="Route11" color="4" fill="7" visible="no" active="no"/>
-<layer number="12" name="Route12" color="1" fill="5" visible="no" active="no"/>
-<layer number="13" name="Route13" color="4" fill="5" visible="no" active="no"/>
-<layer number="14" name="Route14" color="1" fill="6" visible="no" active="no"/>
-<layer number="15" name="Route15" color="4" fill="6" visible="no" active="no"/>
-<layer number="16" name="Bottom" color="1" fill="1" visible="no" active="no"/>
-<layer number="17" name="Pads" color="2" fill="1" visible="no" active="no"/>
-<layer number="18" name="Vias" color="2" fill="1" visible="no" active="no"/>
-<layer number="19" name="Unrouted" color="6" fill="1" visible="no" active="no"/>
-<layer number="20" name="Dimension" color="15" fill="1" visible="no" active="no"/>
-<layer number="21" name="tPlace" color="7" fill="1" visible="no" active="no"/>
-<layer number="22" name="bPlace" color="7" fill="1" visible="no" active="no"/>
-<layer number="23" name="tOrigins" color="15" fill="1" visible="no" active="no"/>
-<layer number="24" name="bOrigins" color="15" fill="1" visible="no" active="no"/>
-<layer number="25" name="tNames" color="7" fill="1" visible="no" active="no"/>
-<layer number="26" name="bNames" color="7" fill="1" visible="no" active="no"/>
-<layer number="27" name="tValues" color="7" fill="1" visible="no" active="no"/>
-<layer number="28" name="bValues" color="7" fill="1" visible="no" active="no"/>
+<layer number="1" name="Top" color="4" fill="1" visible="yes" active="no"/>
+<layer number="2" name="Route2" color="1" fill="3" visible="yes" active="no"/>
+<layer number="3" name="Route3" color="4" fill="3" visible="yes" active="no"/>
+<layer number="4" name="Route4" color="1" fill="4" visible="yes" active="no"/>
+<layer number="5" name="Route5" color="4" fill="4" visible="yes" active="no"/>
+<layer number="6" name="Route6" color="1" fill="8" visible="yes" active="no"/>
+<layer number="7" name="Route7" color="4" fill="8" visible="yes" active="no"/>
+<layer number="8" name="Route8" color="1" fill="2" visible="yes" active="no"/>
+<layer number="9" name="Route9" color="4" fill="2" visible="yes" active="no"/>
+<layer number="10" name="Route10" color="1" fill="7" visible="yes" active="no"/>
+<layer number="11" name="Route11" color="4" fill="7" visible="yes" active="no"/>
+<layer number="12" name="Route12" color="1" fill="5" visible="yes" active="no"/>
+<layer number="13" name="Route13" color="4" fill="5" visible="yes" active="no"/>
+<layer number="14" name="Route14" color="1" fill="6" visible="yes" active="no"/>
+<layer number="15" name="Route15" color="4" fill="6" visible="yes" active="no"/>
+<layer number="16" name="Bottom" color="1" fill="1" visible="yes" active="no"/>
+<layer number="17" name="Pads" color="2" fill="1" visible="yes" active="no"/>
+<layer number="18" name="Vias" color="2" fill="1" visible="yes" active="no"/>
+<layer number="19" name="Unrouted" color="6" fill="1" visible="yes" active="no"/>
+<layer number="20" name="Dimension" color="15" fill="1" visible="yes" active="no"/>
+<layer number="21" name="tPlace" color="7" fill="1" visible="yes" active="no"/>
+<layer number="22" name="bPlace" color="7" fill="1" visible="yes" active="no"/>
+<layer number="23" name="tOrigins" color="15" fill="1" visible="yes" active="no"/>
+<layer number="24" name="bOrigins" color="15" fill="1" visible="yes" active="no"/>
+<layer number="25" name="tNames" color="7" fill="1" visible="yes" active="no"/>
+<layer number="26" name="bNames" color="7" fill="1" visible="yes" active="no"/>
+<layer number="27" name="tValues" color="7" fill="1" visible="yes" active="no"/>
+<layer number="28" name="bValues" color="7" fill="1" visible="yes" active="no"/>
 <layer number="29" name="tStop" color="7" fill="3" visible="no" active="no"/>
 <layer number="30" name="bStop" color="7" fill="6" visible="no" active="no"/>
@@
 <layer number="35" name="tGlue" color="7" fill="4" visible="no" active="no"/>
 <layer number="36" name="bGlue" color="7" fill="5" visible="no" active="no"/>
-<layer number="37" name="tTest" color="7" fill="1" visible="no" active="no"/>
-<layer number="38" name="bTest" color="7" fill="1" visible="no" active="no"/>
+<layer number="37" name="tTest" color="7" fill="1" visible="yes" active="no"/>
+<layer number="38" name="bTest" color="7" fill="1" visible="yes" active="no"/>
 <layer number="39" name="tKeepout" color="4" fill="11" visible="no" active="no"/>
 <layer number="40" name="bKeepout" color="1" fill="11" visible="no" active="no"/>
@@
 <layer number="44" name="Drills" color="7" fill="1" visible="no" active="no"/>
 <layer number="45" name="Holes" color="7" fill="1" visible="no" active="no"/>
-<layer number="46" name="Milling" color="3" fill="1" visible="no" active="no"/>
-<layer number="47" name="Measures" color="7" fill="1" visible="no" active="no"/>
-<layer number="48" name="Document" color="7" fill="1" visible="no" active="no"/>
-<layer number="49" name="Reference" color="7" fill="1" visible="no" active="no"/>
-<layer number="50" name="dxf" color="7" fill="1" visible="no" active="no"/>
-<layer number="51" name="tDocu" color="7" fill="1" visible="no" active="no"/>
-<layer number="52" name="bDocu" color="7" fill="1" visible="no" active="no"/>
-<layer number="53" name="tGND_GNDA" color="7" fill="9" visible="no" active="no"/>
-<layer number="54" name="bGND_GNDA" color="1" fill="9" visible="no" active="no"/>
-<layer number="56" name="wert" color="7" fill="1" visible="no" active="no"/>
-<layer number="57" name="tCAD" color="7" fill="1" visible="no" active="no"/>
+<layer number="46" name="Milling" color="3" fill="1" visible="yes" active="no"/>
+<layer number="47" name="Measures" color="7" fill="1" visible="yes" active="no"/>
+<layer number="48" name="Document" color="7" fill="1" visible="yes" active="no"/>
+<layer number="49" name="Reference" color="7" fill="1" visible="yes" active="no"/>
+<layer number="50" name="dxf" color="7" fill="1" visible="yes" active="no"/>
+<layer number="51" name="tDocu" color="7" fill="1" visible="yes" active="no"/>
+<layer number="52" name="bDocu" color="7" fill="1" visible="yes" active="no"/>
+<layer number="53" name="tGND_GNDA" color="7" fill="9" visible="yes" active="no"/>
+<layer number="54" name="bGND_GNDA" color="1" fill="9" visible="yes" active="no"/>
+<layer number="56" name="wert" color="7" fill="1" visible="yes" active="no"/>
+<layer number="57" name="tCAD" color="7" fill="1" visible="yes" active="no"/>
 <layer number="90" name="Modules" color="5" fill="1" visible="yes" active="yes"/>
 <layer number="91" name="Nets" color="2" fill="1" visible="yes" active="yes"/>
@@
 <part name="GND2" library="supply1" deviceset="GND" device=""/>
 <part name="X3" library="pinhead" deviceset="PINHD-1X2" device=""/>
+<part name="C18" library="HWProgUSB" deviceset="RCL_CPOL-EU" device="E2-5" value="100µ 16V"/>
+<part name="GND11" library="supply1" deviceset="GND" device=""/>
 </parts>
 <sheets>
@@
 <attribute name="VALUE" x="16.51" y="35.56" size="1.778" layer="96" rot="MR0"/>
 </instance>
+<instance part="C18" gate="G$1" x="134.62" y="38.1"/>
+<instance part="GND11" gate="1" x="134.62" y="27.94"/>
 </instances>
 <busses>
@@
 <pinref part="C8" gate="G$1" pin="-"/>
 <wire x1="111.76" y1="30.48" x2="111.76" y2="33.02" width="0.1524" layer="91"/>
+</segment>
+<segment>
+<pinref part="C18" gate="G$1" pin="-"/>
+<pinref part="GND11" gate="1" pin="GND"/>
+<wire x1="134.62" y1="33.02" x2="134.62" y2="30.48" width="0.1524" layer="91"/>
 </segment>
 </net>
@@
 <wire x1="111.76" y1="48.26" x2="121.92" y2="48.26" width="0.1524" layer="91"/>
 <junction x="121.92" y="48.26"/>
+<wire x1="121.92" y1="48.26" x2="134.62" y2="48.26" width="0.1524" layer="91"/>
+<pinref part="C18" gate="G$1" pin="+"/>
+<wire x1="134.62" y1="48.26" x2="134.62" y2="40.64" width="0.1524" layer="91"/>
 </segment>
 </net>
