File: ESR_NM8032.sch (EAGLE design)
At the start: 59 parts, among them IC1 LD117AS12TR

Commit message: ,
Parts:
- added C19: 470x6v3, rcl:CPOL-EUE15-5AXIAL
Changed lines of the file:
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@@
 <part name="GND11" library="supply1" deviceset="GND" device=""/>
 <part name="IC1" library="v-reg" deviceset="LD117A?*" device="S" technology="12TR"/>
+<part name="C19" library="rcl" deviceset="CPOL-EU" device="E15-5AXIAL" value="470x6v3"/>
 </parts>
 <sheets>
@@
 <instance part="GND11" gate="1" x="147.32" y="27.94"/>
 <instance part="IC1" gate="G$1" x="134.62" y="63.5"/>
+<instance part="C19" gate="G$1" x="71.12" y="93.98"/>
 </instances>
 <busses>

Commit message: .
Parts:
- removed IC1: LD117AS12TR, v-reg:LD117AS12TR
- added C20: 100n, rcl:C-EUC0805
- added DA5: (no value), ct-pack:78LXX_SOT89
- C13, C14: device HWProgUSB:RCL_CPOL-EUE3.5-8 -> HWProgUSB:RCL_CPOL-EUE2.5-7
Connections:
- new net VCC/2: C17.1, C8.+, DA5.IN, HL1.A, HL10.A, HL2.A, HL3.A, HL4.A, HL5.A, HL6.A, HL7.A, HL8.A, HL9.A, L3.2
- net GND: now also C17.2, C20.2, DA5.GND; no longer C17.1
- net V+: now also C20.1, DA5.OUT; no longer C17.2, C8.+, HL1.A, HL10.A, HL2.A, HL3.A, HL4.A, HL5.A, HL6.A, HL7.A, HL8.A, HL9.A, L3.2
Other:
- moved on the sheet: C17, C18

Commit message: .
Parts:
- added C21: 100µ 16V, HWProgUSB:RCL_CPOL-EUE2-5
- added C22: 100n, rcl:C-EUC0805
- added C23, C24: 470x6v3, rcl:CPOL-EUE15-5AXIAL
- added H1, H2, H3: MOUNT-PAD-SQUARE3.2, holes:MOUNT-PAD-SQUARE3.2
- R16: device rcl:R-EU_M0805 -> rcl:R-EU_0207/15
- R5: device rcl:R-EU_0207/10 -> rcl:R-EU_0204/7
Connections:
- net GND: now also C21.-, C22.2
- net V+: now also C21.+, C22.1

Commit message: ..
Parts:
- added L2.2: (no value), pinhead:PINHD-1X1
- C13: value 470µ / 10V -> 470µ
Connections:
- removed net N$15: C2.2, C9.-, DD1P.VSS, VD2.A, X1.1
- removed net N$17: C2.1, C9.+, DD1P.VDD, L1.1, VD1.C
- new net GNDS: C19.-, C2.2, C23.-, C24.-, C9.-, DD1P.VSS, VD2.A, X1.1
- new net VCCS: C19.+, C2.1, C23.+, C24.+, C9.+, DD1P.VDD, L1.1, VD1.C
- net N$30: now also L2.2.1
Other:
- moved on the sheet: C19, C23, C24, R13

Commit message: rr1
Parts:
- removed X3: (no value), pinhead:PINHD-1X2
- added U$2: B-, ESR_NM8032:B-
- added U$4: B+, ESR_NM8032:B+
- C2: device rcl:C-EU050-025X075 -> rcl:C-EU075-032X103
- R1: device rcl:R-EU_0207/10 -> rcl:R-EU_M0805
Connections:
- removed net +5V: C12.1, C13.+, DA4.VCC, R13.1, X3.1
- new net N$15: C12.1, C13.+, DA4.VCC, R13.1, U$4.P$1
- net GND: now also U$2.P$1; no longer X3.2

Commit message: .
Parts:
- L2: device rcl:L-US0207/10 -> rcl:L-US0204/7
- L3: device rcl:L-US0207/10 -> rcl:L-US0204/5
- R16: device rcl:R-EU_0207/15 -> rcl:R-EU_M0805
Changed lines of the file:
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@@
 <part name="R13" library="rcl" deviceset="R-EU_" device="M1206" value="0.5-1"/>
 <part name="GND6" library="supply1" deviceset="GND" device=""/>
-<part name="R16" library="rcl" deviceset="R-EU_" device="0207/15" value="9k1"/>
+<part name="R16" library="rcl" deviceset="R-EU_" device="M0805" value="9k1"/>
 <part name="R15" library="rcl" deviceset="R-EU_" device="M0805" value="2k4"/>
-<part name="L2" library="rcl" deviceset="L-US" device="0207/10" value="100uh"/>
+<part name="L2" library="rcl" deviceset="L-US" device="0204/7" value="100uh"/>
 <part name="3VD2" library="diode" deviceset="SCHOTTKY-DIODE" device="SMD" value="SS12"/>
 <part name="C16" library="rcl" deviceset="C-EU" device="C0805" value="1n"/>
@@
 <part name="C9" library="rcl" deviceset="CPOL-EU" device="E15-5AXIAL" value="470x6v3"/>
 <part name="C10" library="rcl" deviceset="C-EU" device="C0805" value="330n"/>
-<part name="L3" library="rcl" deviceset="L-US" device="0207/10" value="100uh"/>
+<part name="L3" library="rcl" deviceset="L-US" device="0204/5" value="100uh"/>
 <part name="P+1" library="supply1" deviceset="V+" device=""/>
 <part name="DA2" library="ESR_NM8032" deviceset="K157DA1" device=""/>

Commit message: .,
Parts:
- added SW2, SW3: (no value), pinhead:PINHD-1X3
Connections:
- new net N$17: SW2.1, U$4.P$1
- new net N$27: SW3.3, U$2.P$1
- net GND: now also SW3.2; no longer U$2.P$1
- net N$15: now also SW2.2; no longer U$4.P$1
Changed lines of the file:
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@@
 <grid distance="100" unitdist="mil" unit="mil" style="lines" multiple="1" display="yes" altdistance="0.01" altunitdist="inch" altunit="inch"/>
 <layers>
-<layer number="1" name="Top" color="4" fill="1" visible="yes" active="no"/>
-<layer number="2" name="Route2" color="1" fill="3" visible="yes" active="no"/>
-<layer number="3" name="Route3" color="4" fill="3" visible="yes" active="no"/>
-<layer number="4" name="Route4" color="1" fill="4" visible="yes" active="no"/>
-<layer number="5" name="Route5" color="4" fill="4" visible="yes" active="no"/>
-<layer number="6" name="Route6" color="1" fill="8" visible="yes" active="no"/>
-<layer number="7" name="Route7" color="4" fill="8" visible="yes" active="no"/>
-<layer number="8" name="Route8" color="1" fill="2" visible="yes" active="no"/>
-<layer number="9" name="Route9" color="4" fill="2" visible="yes" active="no"/>
-<layer number="10" name="Route10" color="1" fill="7" visible="yes" active="no"/>
-<layer number="11" name="Route11" color="4" fill="7" visible="yes" active="no"/>
-<layer number="12" name="Route12" color="1" fill="5" visible="yes" active="no"/>
-<layer number="13" name="Route13" color="4" fill="5" visible="yes" active="no"/>
-<layer number="14" name="Route14" color="1" fill="6" visible="yes" active="no"/>
-<layer number="15" name="Route15" color="4" fill="6" visible="yes" active="no"/>
-<layer number="16" name="Bottom" color="1" fill="1" visible="yes" active="no"/>
-<layer number="17" name="Pads" color="2" fill="1" visible="yes" active="no"/>
-<layer number="18" name="Vias" color="2" fill="1" visible="yes" active="no"/>
-<layer number="19" name="Unrouted" color="6" fill="1" visible="yes" active="no"/>
-<layer number="20" name="Dimension" color="15" fill="1" visible="yes" active="no"/>
-<layer number="21" name="tPlace" color="7" fill="1" visible="yes" active="no"/>
-<layer number="22" name="bPlace" color="7" fill="1" visible="yes" active="no"/>
-<layer number="23" name="tOrigins" color="15" fill="1" visible="yes" active="no"/>
-<layer number="24" name="bOrigins" color="15" fill="1" visible="yes" active="no"/>
-<layer number="25" name="tNames" color="7" fill="1" visible="yes" active="no"/>
-<layer number="26" name="bNames" color="7" fill="1" visible="yes" active="no"/>
-<layer number="27" name="tValues" color="7" fill="1" visible="yes" active="no"/>
-<layer number="28" name="bValues" color="7" fill="1" visible="yes" active="no"/>
+<layer number="1" name="Top" color="4" fill="1" visible="no" active="no"/>
+<layer number="2" name="Route2" color="1" fill="3" visible="no" active="no"/>
+<layer number="3" name="Route3" color="4" fill="3" visible="no" active="no"/>
+<layer number="4" name="Route4" color="1" fill="4" visible="no" active="no"/>
+<layer number="5" name="Route5" color="4" fill="4" visible="no" active="no"/>
+<layer number="6" name="Route6" color="1" fill="8" visible="no" active="no"/>
+<layer number="7" name="Route7" color="4" fill="8" visible="no" active="no"/>
+<layer number="8" name="Route8" color="1" fill="2" visible="no" active="no"/>
+<layer number="9" name="Route9" color="4" fill="2" visible="no" active="no"/>
+<layer number="10" name="Route10" color="1" fill="7" visible="no" active="no"/>
+<layer number="11" name="Route11" color="4" fill="7" visible="no" active="no"/>
+<layer number="12" name="Route12" color="1" fill="5" visible="no" active="no"/>
+<layer number="13" name="Route13" color="4" fill="5" visible="no" active="no"/>
+<layer number="14" name="Route14" color="1" fill="6" visible="no" active="no"/>
+<layer number="15" name="Route15" color="4" fill="6" visible="no" active="no"/>
+<layer number="16" name="Bottom" color="1" fill="1" visible="no" active="no"/>
+<layer number="17" name="Pads" color="2" fill="1" visible="no" active="no"/>
+<layer number="18" name="Vias" color="2" fill="1" visible="no" active="no"/>
+<layer number="19" name="Unrouted" color="6" fill="1" visible="no" active="no"/>
+<layer number="20" name="Dimension" color="15" fill="1" visible="no" active="no"/>
+<layer number="21" name="tPlace" color="7" fill="1" visible="no" active="no"/>
+<layer number="22" name="bPlace" color="7" fill="1" visible="no" active="no"/>
+<layer number="23" name="tOrigins" color="15" fill="1" visible="no" active="no"/>
+<layer number="24" name="bOrigins" color="15" fill="1" visible="no" active="no"/>
+<layer number="25" name="tNames" color="7" fill="1" visible="no" active="no"/>
+<layer number="26" name="bNames" color="7" fill="1" visible="no" active="no"/>
+<layer number="27" name="tValues" color="7" fill="1" visible="no" active="no"/>
+<layer number="28" name="bValues" color="7" fill="1" visible="no" active="no"/>
 <layer number="29" name="tStop" color="7" fill="3" visible="no" active="no"/>
 <layer number="30" name="bStop" color="7" fill="6" visible="no" active="no"/>
@@
 <layer number="35" name="tGlue" color="7" fill="4" visible="no" active="no"/>
 <layer number="36" name="bGlue" color="7" fill="5" visible="no" active="no"/>
-<layer number="37" name="tTest" color="7" fill="1" visible="yes" active="no"/>
-<layer number="38" name="bTest" color="7" fill="1" visible="yes" active="no"/>
+<layer number="37" name="tTest" color="7" fill="1" visible="no" active="no"/>
+<layer number="38" name="bTest" color="7" fill="1" visible="no" active="no"/>
 <layer number="39" name="tKeepout" color="4" fill="11" visible="no" active="no"/>
 <layer number="40" name="bKeepout" color="1" fill="11" visible="no" active="no"/>
@@
 <layer number="44" name="Drills" color="7" fill="1" visible="no" active="no"/>
 <layer number="45" name="Holes" color="7" fill="1" visible="no" active="no"/>
-<layer number="46" name="Milling" color="3" fill="1" visible="yes" active="no"/>
-<layer number="47" name="Measures" color="7" fill="1" visible="yes" active="no"/>
-<layer number="48" name="Document" color="7" fill="1" visible="yes" active="no"/>
-<layer number="49" name="Reference" color="7" fill="1" visible="yes" active="no"/>
-<layer number="50" name="dxf" color="7" fill="1" visible="yes" active="no"/>
-<layer number="51" name="tDocu" color="7" fill="1" visible="yes" active="no"/>
-<layer number="52" name="bDocu" color="7" fill="1" visible="yes" active="no"/>
-<layer number="53" name="tGND_GNDA" color="7" fill="9" visible="yes" active="no"/>
-<layer number="54" name="bGND_GNDA" color="1" fill="9" visible="yes" active="no"/>
-<layer number="56" name="wert" color="7" fill="1" visible="yes" active="no"/>
-<layer number="57" name="tCAD" color="7" fill="1" visible="yes" active="no"/>
+<layer number="46" name="Milling" color="3" fill="1" visible="no" active="no"/>
+<layer number="47" name="Measures" color="7" fill="1" visible="no" active="no"/>
+<layer number="48" name="Document" color="7" fill="1" visible="no" active="no"/>
+<layer number="49" name="Reference" color="7" fill="1" visible="no" active="no"/>
+<layer number="50" name="dxf" color="7" fill="1" visible="no" active="no"/>
+<layer number="51" name="tDocu" color="7" fill="1" visible="no" active="no"/>
+<layer number="52" name="bDocu" color="7" fill="1" visible="no" active="no"/>
+<layer number="53" name="tGND_GNDA" color="7" fill="9" visible="no" active="no"/>
+<layer number="54" name="bGND_GNDA" color="1" fill="9" visible="no" active="no"/>
+<layer number="56" name="wert" color="7" fill="1" visible="no" active="no"/>
+<layer number="57" name="tCAD" color="7" fill="1" visible="no" active="no"/>
 <layer number="90" name="Modules" color="5" fill="1" visible="yes" active="yes"/>
 <layer number="91" name="Nets" color="2" fill="1" visible="yes" active="yes"/>
@@
 <part name="U$2" library="ESR_NM8032" deviceset="B-" device=""/>
 <part name="U$4" library="ESR_NM8032" deviceset="B+" device=""/>
+<part name="SW2" library="pinhead" deviceset="PINHD-1X3" device=""/>
+<part name="SW3" library="pinhead" deviceset="PINHD-1X3" device=""/>
 </parts>
 <sheets>
@@
 <instance part="U$2" gate="G$1" x="22.86" y="40.64"/>
 <instance part="U$4" gate="G$1" x="22.86" y="48.26"/>
+<instance part="SW2" gate="A" x="12.7" y="55.88" rot="R180"/>
+<instance part="SW3" gate="A" x="12.7" y="30.48" rot="R180"/>
 </instances>
 <busses>
@@
 <wire x1="38.1" y1="39.37" x2="38.1" y2="27.94" width="0.1524" layer="91"/>
 <junction x="38.1" y="27.94"/>
-<pinref part="U$2" gate="G$1" pin="P$1"/>
-<wire x1="22.86" y1="38.1" x2="22.86" y2="27.94" width="0.1524" layer="91"/>
+<wire x1="22.86" y1="30.48" x2="22.86" y2="27.94" width="0.1524" layer="91"/>
 <wire x1="30.48" y1="27.94" x2="22.86" y2="27.94" width="0.1524" layer="91"/>
+<pinref part="SW3" gate="A" pin="2"/>
+<wire x1="15.24" y1="30.48" x2="22.86" y2="30.48" width="0.1524" layer="91"/>
 </segment>
 <segment>
@@
 <pinref part="C13" gate="G$1" pin="+"/>
 <wire x1="38.1" y1="46.99" x2="38.1" y2="55.88" width="0.1524" layer="91"/>
-<wire x1="22.86" y1="55.88" x2="30.48" y2="55.88" width="0.1524" layer="91"/>
-<wire x1="22.86" y1="50.8" x2="22.86" y2="55.88" width="0.1524" layer="91"/>
 <wire x1="30.48" y1="60.96" x2="30.48" y2="55.88" width="0.1524" layer="91"/>
+<pinref part="SW2" gate="A" pin="2"/>
+<wire x1="15.24" y1="55.88" x2="30.48" y2="55.88" width="0.1524" layer="91"/>
+</segment>
+</net>
+<net name="N$17" class="0">
+<segment>
 <pinref part="U$4" gate="G$1" pin="P$1"/>
-</segment>
-</net>
+<wire x1="22.86" y1="50.8" x2="22.86" y2="53.34" width="0.1524" layer="91"/>
+<pinref part="SW2" gate="A" pin="1"/>
+<wire x1="15.24" y1="53.34" x2="22.86" y2="53.34" width="0.1524" layer="91"/>
+</segment>
+</net>
+<net name="N$27" class="0">
+<segment>
+<pinref part="U$2" gate="G$1" pin="P$1"/>
+<wire x1="22.86" y1="38.1" x2="22.86" y2="33.02" width="0.1524" layer="91"/>
+<pinref part="SW3" gate="A" pin="3"/>
+<wire x1="15.24" y1="33.02" x2="22.86" y2="33.02" width="0.1524" layer="91"/>
+</segment>
+</net>

Commit message: .
Parts:
- removed C19, C23, C24: 470x6v3, rcl:CPOL-EUE15-5AXIAL
Connections:
- net GNDS: no longer C19.-, C23.-, C24.-
- net VCCS: no longer C19.+, C23.+, C24.+
Changed lines of the file:
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@@
 <part name="C18" library="HWProgUSB" deviceset="RCL_CPOL-EU" device="E2-5" value="100µ 16V"/>
 <part name="GND11" library="supply1" deviceset="GND" device=""/>
-<part name="C19" library="rcl" deviceset="CPOL-EU" device="E15-5AXIAL" value="470x6v3"/>
 <part name="DA5" library="ct-pack" deviceset="78LXX" device="_SOT89"/>
 <part name="GND12" library="supply1" deviceset="GND" device=""/>
@@
 <part name="H2" library="holes" deviceset="MOUNT-PAD-SQUARE" device="3.2"/>
 <part name="H3" library="holes" deviceset="MOUNT-PAD-SQUARE" device="3.2"/>
-<part name="C23" library="rcl" deviceset="CPOL-EU" device="E15-5AXIAL" value="470x6v3"/>
-<part name="C24" library="rcl" deviceset="CPOL-EU" device="E15-5AXIAL" value="470x6v3"/>
 <part name="L2.2" library="pinhead" deviceset="PINHD-1X1" device=""/>
 <part name="U$2" library="ESR_NM8032" deviceset="B-" device=""/>
@@
 <instance part="C18" gate="G$1" x="142.24" y="38.1"/>
 <instance part="GND11" gate="1" x="142.24" y="27.94"/>
-<instance part="C19" gate="G$1" x="12.7" y="175.26"/>
 <instance part="DA5" gate="1" x="132.08" y="63.5"/>
 <instance part="GND12" gate="1" x="132.08" y="50.8"/>
@@
 <instance part="H2" gate="G$1" x="177.8" y="73.66"/>
 <instance part="H3" gate="G$1" x="177.8" y="66.04"/>
-<instance part="C23" gate="G$1" x="25.4" y="175.26"/>
-<instance part="C24" gate="G$1" x="38.1" y="175.26"/>
 <instance part="L2.2" gate="G$1" x="41.91" y="71.12" smashed="yes" rot="R90">
 <attribute name="NAME" x="39.37" y="73.025" size="1.778" layer="95"/>
@@
 <label x="71.12" y="124.46" size="1.778" layer="95"/>
 </segment>
-<segment>
-<pinref part="C19" gate="G$1" pin="-"/>
-<wire x1="12.7" y1="170.18" x2="12.7" y2="167.64" width="0.1524" layer="91"/>
-<wire x1="12.7" y1="167.64" x2="25.4" y2="167.64" width="0.1524" layer="91"/>
-<pinref part="C23" gate="G$1" pin="-"/>
-<wire x1="25.4" y1="167.64" x2="25.4" y2="170.18" width="0.1524" layer="91"/>
-<pinref part="C24" gate="G$1" pin="-"/>
-<wire x1="25.4" y1="167.64" x2="38.1" y2="167.64" width="0.1524" layer="91"/>
-<wire x1="38.1" y1="167.64" x2="38.1" y2="170.18" width="0.1524" layer="91"/>
-<label x="27.94" y="165.1" size="1.778" layer="95"/>
-<junction x="25.4" y="167.64"/>
-</segment>
 </net>
 <net name="VCCS" class="0">
@@
 <label x="71.12" y="142.24" size="1.778" layer="95"/>
 </segment>
-<segment>
-<pinref part="C24" gate="G$1" pin="+"/>
-<wire x1="25.4" y1="180.34" x2="38.1" y2="180.34" width="0.1524" layer="91"/>
-<wire x1="38.1" y1="180.34" x2="38.1" y2="177.8" width="0.1524" layer="91"/>
-<pinref part="C19" gate="G$1" pin="+"/>
-<wire x1="12.7" y1="177.8" x2="12.7" y2="180.34" width="0.1524" layer="91"/>
-<wire x1="12.7" y1="180.34" x2="25.4" y2="180.34" width="0.1524" layer="91"/>
-<pinref part="C23" gate="G$1" pin="+"/>
-<wire x1="25.4" y1="180.34" x2="25.4" y2="177.8" width="0.1524" layer="91"/>
-<label x="27.94" y="180.34" size="1.778" layer="95"/>
-<junction x="25.4" y="180.34"/>
-</segment>
-</net>
+</net>
