File: ESR_NM8032.brd (EAGLE design)
At the start: 34.9 x 91.4 mm, 74 parts

Commit message: .
Parts:
- removed C19, C23, C24: 470x6v3, rcl:E15-5
- moved C9 88.9 mm to (-11.7, 39.4)
- moved R5 2.56 mm to (12.4, 49.5)
- moved R2 2.48 mm to (21.3, 48.9), turned to 270 degrees
- moved R3 2.25 mm to (20.6, 45.4)
- moved SW1 1.93 mm to (24.4, 47.9)
- moved C4 1.35 mm to (19.1, 41.0)
- moved L1 0.32 mm to (16.5, 40.6)
Connections:
- net GNDS: no longer C19.-, C23.-, C24.-
- net VCCS: no longer C19.+, C23.+, C24.+
Routing:
- net GND: track 281.0 -> 284.7 mm
- net N$27: track 24.4 -> 28.0 mm

Commit message: .
Parts:
- moved C14 28.3 mm to (-16.5, 116.2)
- moved C15 22.9 mm to (-15.6, 110.8)
- moved 3VD2 17.6 mm to (23.8, 112.1)
- moved R16 9.34 mm to (17.8, 99.1)
- moved C12 3.24 mm to (14.0, 102.9), turned to 180 degrees
- moved C13 2.54 mm to (14.3, 105.1)
- moved L3 2.25 mm to (5.40, 100.6), turned to 270 degrees
Routing:
- net GND: track 284.7 -> 261.6 mm
- net N$15: track 13.4 -> 10.1 mm

Commit message: p2k
Parts:
- added S1, S2: П2К, ESR_NM8032:P2K
- moved R5 13.4 mm to (-0.32, 53.7)
- moved SW1 4.42 mm to (26.0, 52.1)
- moved R2 4.32 mm to (22.5, 53.0)
- moved R3 3.55 mm to (22.2, 48.6)
- moved C5 0.90 mm to (6.67, 65.7), turned to 90 degrees
- moved R7 0.90 mm to (6.67, 61.6)
Connections:
- new net N$28: S1.S2B, S2.S1B
- new net N$39: S1.S2, S2.S1
Routing:
- net GND: track 261.6 -> 279.1 mm, vias 2 -> 0
- net N$37: track 33.5 -> 32.4 mm
Other:
- board size 34.9 x 91.4 mm -> 34.9 x 91.7 mm

Commit message: ,n
Parts:
- moved S1 12.1 mm to (23.8, 28.6), turned to 180 degrees
- moved C9 11.3 mm to (-17.8, 48.9)
- moved S2 9.61 mm to (11.4, 28.9), turned to 180 degrees
- moved C1 5.65 mm to (0.95, 36.2), turned to 180 degrees
- moved L1 5.32 mm to (14.9, 45.7), turned to 0 degrees
- moved C2 4.96 mm to (6.99, 42.9)
- moved VD2 3.38 mm to (9.21, 40.0)
- moved VD1 3.18 mm to (9.21, 42.2)
- moved DD1 3.14 mm to (0.95, 42.2)
- moved C3 2.42 mm to (4.76, 48.6)
- moved R3 1.91 mm to (22.2, 50.5)
- moved R2 1.59 mm to (22.5, 54.6)
- moved SW1 0.95 mm to (26.0, 53.0)
- moved R1 0.71 mm to (-2.86, 36.2), turned to 0 degrees
- moved U$1 0.32 mm to (-1.59, 47.6)
Routing:
- net GNDS: track 13.1 -> 16.7 mm
- net N$1: track 27.3 -> 24.1 mm
- net N$4: track 10.7 -> 7.94 mm
- net N$2: track 43.4 -> 40.6 mm
- net N$6: track 2.72 -> 0.00 mm
Other:
- board size 34.9 x 91.7 mm -> 34.9 x 93.3 mm

Commit message: ,
Parts:
- moved S2 37.6 mm to (48.9, 32.4), turned to 270 degrees
- moved S1 35.1 mm to (50.2, 51.8), turned to 270 degrees
Changed lines of the file:
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@@
 </element>
 <element name="X2" library="pinhead" package="1X02" value="" x="25.0825" y="40.64" smashed="yes" rot="R180">
-<attribute name="NAME" x="24.0538" y="37.3888" size="1.27" layer="25" ratio="10"/>
+<attribute name="NAME" x="25.6413" y="37.7063" size="1.27" layer="25" ratio="10"/>
 <attribute name="VALUE" x="27.6225" y="43.815" size="1.27" layer="27" rot="R180"/>
 </element>
@@
 <element name="SW2" library="pinhead" package="1X03" value="" x="7.9375" y="118.745"/>
 <element name="SW3" library="pinhead" package="1X03" value="" x="25.0825" y="29.5275" rot="R270"/>
-<element name="S1" library="ESR_NM8032" package="P2K" value="П2К" x="23.8125" y="28.575" rot="R180"/>
-<element name="S2" library="ESR_NM8032" package="P2K" value="П2К" x="11.43" y="28.8925" rot="R180"/>
+<element name="S1" library="ESR_NM8032" package="P2K" value="П2К" x="50.165" y="51.7525" rot="R270"/>
+<element name="S2" library="ESR_NM8032" package="P2K" value="П2К" x="48.895" y="32.385" rot="R270"/>
 </elements>
 <signals>
@@
 <contactref element="S1" pad="S2B"/>
 <contactref element="S2" pad="S1B"/>
-<wire x1="14.48" y1="40.5125" x2="20.7625" y2="40.195" width="0" layer="19" extent="1-1"/>
+<wire x1="37.275" y1="35.435" x2="38.545" y2="48.7025" width="0" layer="19" extent="1-1"/>
 </signal>
 <signal name="N$39">
 <contactref element="S2" pad="S1"/>
 <contactref element="S1" pad="S2"/>
-<wire x1="14.48" y1="36.5125" x2="20.7625" y2="36.195" width="0" layer="19" extent="1-1"/>
+<wire x1="41.275" y1="35.435" x2="42.545" y2="48.7025" width="0" layer="19" extent="1-1"/>
 </signal>
 </signals>

Commit message: 1
Parts:
- removed S1, S2: П2К, ESR_NM8032:P2K
- removed SW1, SW2, SW3: (no value), pinhead:1X03
- added JP2, POWER_ON: (no value), pinhead:2X03
- moved R3 8.03 mm to (19.7, 42.9)
- moved R2 6.48 mm to (21.3, 48.3)
- moved H2 6.33 mm to (28.9, 121.3)
- moved C4 3.81 mm to (15.2, 41.0)
- moved X2 1.35 mm to (24.1, 39.7)
Connections:
- removed net N$15: C12.1, C13.+, DA4.6, R13.1, SW2.2
- removed net N$17: SW2.1, U$4.P$1
- removed net N$28: S1.S2B, S2.S1B
- removed net N$39: S1.S2, S2.S1
- new net +6V: C12.1, C13.+, DA4.6, R13.1, U$4.P$1
- net GND: now also POWER_ON.3, POWER_ON.4; no longer SW3.2
- net N$16: now also JP2.3, JP2.4; no longer SW1.2
- net N$23: now also JP2.1, JP2.2; no longer SW1.3
- net N$25: now also JP2.5, JP2.6; no longer SW1.1
- net N$27: now also POWER_ON.1, POWER_ON.2; no longer SW3.3
Routing:
- net N$15: track 10.1 -> 0.00 mm
- net +6V: track 0.00 -> 10.1 mm
- net GND: track 279.1 -> 276.6 mm
- net N$27: track 28.0 -> 25.8 mm

Commit message: .
Parts:
- moved C9 34.1 mm to (14.0, 36.5)
Changed lines of the file:
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@@
 <attribute name="VALUE" x="12.6619" y="45.085" size="1.27" layer="27" ratio="10"/>
 </element>
-<element name="C9" library="rcl" package="E15-5" value="470x6v3" x="-17.78" y="48.895" smashed="yes" rot="R270">
-<attribute name="NAME" x="-18.3515" y="46.609" size="1.27" layer="25" ratio="10" rot="R90"/>
-<attribute name="VALUE" x="-16.1798" y="44.069" size="1.27" layer="27" ratio="10" rot="R90"/>
+<element name="C9" library="rcl" package="E15-5" value="470x6v3" x="13.97" y="36.5125" smashed="yes" rot="R270">
+<attribute name="NAME" x="13.3985" y="34.2265" size="1.27" layer="25" ratio="10" rot="R90"/>
+<attribute name="VALUE" x="15.5702" y="31.6865" size="1.27" layer="27" ratio="10" rot="R90"/>
 </element>
 <element name="C10" library="rcl" package="C0805" value="330n" x="14.2875" y="55.5625" rot="MR0"/>
@@
 <wire x1="9.2075" y1="38.4175" x2="6.985" y2="39.0525" width="0.6096" layer="16"/>
 <wire x1="6.985" y1="39.0525" x2="10.16" y2="31.4325" width="0.6096" layer="16"/>
-<wire x1="-17.78" y1="41.275" x2="4.0259" y2="37.7825" width="0" layer="19" extent="16-16"/>
+<wire x1="10.16" y1="31.4325" x2="13.97" y2="28.8925" width="0" layer="19" extent="1-1"/>
 </signal>
 <signal name="VCCS">
@@
 <wire x1="9.8425" y1="45.4025" x2="10.9075" y2="43.7025" width="0.6096" layer="16"/>
 <wire x1="10.9075" y1="43.7025" x2="10.9075" y2="42.2275" width="0.6096" layer="16"/>
-<wire x1="9.8425" y1="45.4025" x2="9.8425" y2="45.72" width="0" layer="19" extent="16-16"/>
-<wire x1="-17.78" y1="56.515" x2="4.0259" y2="46.6725" width="0" layer="19" extent="16-16"/>
+<wire x1="10.9075" y1="43.7025" x2="13.97" y2="44.1325" width="0" layer="19" extent="16-16"/>
+<wire x1="9.8425" y1="45.72" x2="9.8425" y2="45.4025" width="0" layer="19" extent="16-16"/>
 </signal>
 <signal name="N$18">

Commit message: .
Parts:
- removed JP2, POWER_ON: (no value), pinhead:2X03
- added C19: 470x6v3, rcl:E15-5
- added R17: 3k, rcl:R0805
- added S1, S2: (no value), ESR_NM8032:SWITCH9X4
- R5: device rcl:0204/7 -> rcl:M0805
- moved H1 68.1 mm to (6.67, 16.2)
- moved H3 45.5 mm to (-22.2, 57.5)
- moved C14 28.3 mm to (7.30, 101.0), turned to 90 degrees
- moved C15 27.3 mm to (9.53, 100.0), turned to 270 degrees
- moved R5 17.3 mm to (16.8, 51.1), flipped to the bottom, turned to 0 degrees
- moved C5 14.9 mm to (6.35, 50.8), turned to 180 degrees
- moved C4 14.2 mm to (24.1, 52.1)
- moved R16 12.5 mm to (21.0, 111.1), turned to 180 degrees
- moved R4 11.4 mm to (19.4, 60.6), turned to 90 degrees
- moved R6 10.5 mm to (17.8, 53.7), turned to 180 degrees
- moved R2 10.1 mm to (19.1, 38.4), turned to 0 degrees
- moved L3 9.67 mm to (14.3, 96.8), turned to 180 degrees
- moved C6 9.57 mm to (16.8, 53.7), turned to 0 degrees
- moved X2 8.98 mm to (25.4, 48.6), turned to 90 degrees
- moved R7 8.72 mm to (8.26, 53.0), turned to 180 degrees
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Connections:
- removed net N$27: POWER_ON.1, POWER_ON.2, U$2.P$1
- new net N$28: HL1.A, HL10.A, HL2.A, HL3.A, HL4.A, HL5.A, HL6.A, HL7.A, HL8.A, HL9.A, R17.2
- new net N$40: R3.1, S2.11, S2.21
- new net N$42: R2.1, S2.12, S2.22
- net GND: now also S1.10, S1.20; no longer POWER_ON.3, POWER_ON.4
- net GNDS: now also C19.-
- net N$16: now also S2.10, S2.20; no longer JP2.3, JP2.4
- net N$23: now also S1.12, S1.22, U$2.P$1; no longer JP2.1, JP2.2, R3.1
- net N$25: now also S1.11, S1.21; no longer JP2.5, JP2.6, R2.1
- net VCC/2: now also R17.1; no longer HL1.A, HL10.A, HL2.A, HL3.A, HL4.A, HL5.A, HL6.A, HL7.A, HL8.A, HL9.A
- net VCCS: now also C19.+
Routing:
- net N$28: track 0.00 -> 65.1 mm
- net VCC/2: track 82.7 -> 22.0 mm
- net N$38: track 0.00 -> 31.1 mm
- net N$27: track 25.8 -> 0.00 mm
- net N$23: track 0.00 -> 24.7 mm
- net +6V: track 10.1 -> 33.4 mm
- net N$26: track 0.00 -> 22.5 mm
- net N$24: track 51.1 -> 31.5 mm
- net V+: track 87.4 -> 73.1 mm
- net GND: track 276.6 -> 288.1 mm
- net N$33: track 2.19 -> 12.3 mm
- net GNDS: track 16.7 -> 25.7 mm
- net VCCS: track 9.57 -> 15.9 mm
- net N$29: track 0.00 -> 6.11 mm
- net N$22: track 0.00 -> 5.49 mm
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Other:
- board size 34.9 x 93.3 mm -> 34.9 x 90.8 mm
