File: ESR_NM8032.brd (EAGLE design)
At the start: 34.9 x 90.8 mm, 72 parts

Commit message: pcspl
Parts:
- removed H1, H2, H3: MOUNT-PAD-SQUARE3.2, holes:3,2-PAD-SQUARE
- DA5: value (none) -> 78l06
- moved C4 7.25 mm to (17.5, 49.2)
- moved L1 1.31 mm to (16.2, 48.9)
- moved R5 1.00 mm to (15.9, 51.4), turned to 180 degrees
- moved R7 0.71 mm to (8.57, 53.7)
- moved C5 0.64 mm to (6.35, 51.4)
- moved C21 0.45 mm to (6.35, 86.7)
- moved X2 0.45 mm to (25.1, 48.3), turned to 180 degrees
- moved DA2 0.32 mm to (14.3, 61.0)
- moved X1 0.32 mm to (6.03, 34.0)
Routing:
- net N$16: track 3.18 -> 12.7 mm
- net V+: track 73.1 -> 80.4 mm
- net GND: track 288.1 -> 294.0 mm
- net N$19: track 2.25 -> 7.29 mm
- net VCCS: track 15.9 -> 20.9 mm
- net N$23: track 24.7 -> 28.8 mm
- net VCC/2: track 22.0 -> 19.7 mm
- net N$22: track 5.49 -> 3.26 mm
- net N$26: track 22.5 -> 24.6 mm
- net N$18: track 8.67 -> 8.04 mm
Other:
- board text added: "+"
- board text added: "-"
- board text added: "6V"

Commit message: ,
Parts:
- added R18: 0, rcl:R1206W
- moved C11 5.17 mm to (8.26, 87.0)
- moved R11 2.71 mm to (13.3, 78.1), turned to 270 degrees
- moved R17 1.00 mm to (12.7, 94.0)
Connections:
- new net N$41: C10.1, C18.+, C20.1, DA2.11, DA3.9, L1.2, R12.2, R18.1, R4.2
- net V+: now also R18.2; no longer C10.1, C18.+, C20.1, DA2.11, DA3.9, L1.2, R12.2, R4.2
Routing:
- net V+: track 80.4 -> 18.2 mm, vias 2 -> 0
- net N$41: track 0.00 -> 61.1 mm
- net N$20: track 2.86 -> 4.08 mm
- net N$28: track 65.1 -> 64.0 mm
- net N$2: track 38.2 -> 37.5 mm

Commit message: `
Parts:
- R17: value 3k -> 10
- moved R17 20.2 mm to (27.0, 108.3), turned to 270 degrees
- moved C14 13.7 mm to (19.1, 108.0), turned to 180 degrees
- moved C15 11.3 mm to (19.1, 106.0), turned to 180 degrees
- moved R13 7.33 mm to (6.03, 107.3), turned to 90 degrees
- moved R16 5.72 mm to (16.2, 114.3)
- moved 3VD2 3.82 mm to (21.9, 111.4), turned to 0 degrees
- moved L2 2.56 mm to (10.5, 110.5)
- moved C12 2.56 mm to (10.5, 100.3)
- moved C13 2.56 mm to (11.7, 102.9)
- moved DA4 2.56 mm to (11.4, 107.0)
- moved L2.2 2.56 mm to (10.5, 112.7)
- moved R14 2.56 mm to (9.53, 110.8)
- moved C16 2.56 mm to (15.2, 102.2)
- moved R15 2.29 mm to (5.71, 114.3), turned to 180 degrees
- moved L3 1.42 mm to (15.6, 97.5), turned to 225 degrees
- renumbered R18 to J1
Routing:
- net N$28: track 64.0 -> 42.2 mm
- net VCC/2: track 19.8 -> 40.8 mm
- net +6V: track 33.4 -> 25.5 mm
- net N$38: track 31.2 -> 25.0 mm
- net GND: track 293.7 -> 299.1 mm
- net N$33: track 12.3 -> 8.01 mm
- net N$31: track 9.60 -> 7.51 mm
- net N$32: track 27.3 -> 26.2 mm, vias 2 -> 0
- net N$41: track 61.1 -> 60.4 mm
- net N$34: track 5.21 -> 5.73 mm

Commit message: .
Parts:
- added R18, R19, R20, R21, R22, R23, R24, R25, R26, R27: 1*, rcl:R0805
- moved R8 0.71 mm to (8.26, 61.9)
- moved C10 0.32 mm to (14.3, 61.0)
Connections:
- new net N$27: DA3.1, R18.1
- new net N$39: DA3.18, R19.1
- new net N$43: DA3.17, R20.1
- new net N$44: DA3.16, R21.1
- new net N$45: DA3.15, R22.1
- new net N$46: DA3.14, R23.1
- new net N$47: DA3.13, R24.1
- new net N$48: DA3.12, R25.1
- new net N$49: DA3.11, R26.1
- new net N$50: DA3.10, R27.1
- net N$10: now also R23.2; no longer DA3.14
- net N$11: now also R24.2; no longer DA3.13
- net N$12: now also R25.2; no longer DA3.12
- net N$13: now also R26.2; no longer DA3.11
- net N$14: now also R27.2; no longer DA3.10
- net N$3: now also R18.2; no longer DA3.1
- net N$5: now also R19.2; no longer DA3.18
- net N$7: now also R20.2; no longer DA3.17
- net N$8: now also R21.2; no longer DA3.16
- net N$9: now also R22.2; no longer DA3.15
Routing:
- net N$3: track 23.4 -> 16.9 mm
- net N$5: track 13.4 -> 6.95 mm
- net N$7: track 11.7 -> 5.68 mm
- net N$39: track 0.00 -> 4.73 mm
- net N$13: track 7.80 -> 3.20 mm
- net N$14: track 9.52 -> 5.05 mm
- net N$12: track 7.01 -> 2.57 mm
- net N$11: track 6.48 -> 2.04 mm
- net N$43: track 0.00 -> 4.28 mm
- net N$10: track 7.27 -> 3.01 mm
- net N$8: track 9.78 -> 5.82 mm
- net N$27: track 0.00 -> 3.33 mm
- net N$9: track 8.06 -> 4.73 mm
- net N$49: track 0.00 -> 3.25 mm
- net N$44: track 0.00 -> 3.18 mm
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
Commit message: .
Parts:
- moved R19 7.68 mm to (14.6, 90.8), turned to 0 degrees
- moved R18 2.93 mm to (11.1, 93.3)
- moved R17 1.42 mm to (25.7, 107.6), turned to 180 degrees
- moved R16 1.27 mm to (14.9, 114.3)
- moved R27 1.14 mm to (21.6, 67.9)
- moved R26 0.45 mm to (21.6, 72.4)
- moved R22 0.32 mm to (21.6, 83.5)
Routing:
- net N$5: track 6.95 -> 16.4 mm
- net VCC/2: track 40.8 -> 38.0 mm
- net N$3: track 16.9 -> 19.4 mm
- net N$39: track 4.73 -> 2.54 mm
- net N$32: track 26.2 -> 25.0 mm
- net N$38: track 25.0 -> 26.3 mm
- net N$50: track 2.56 -> 3.69 mm
- net N$14: track 5.05 -> 3.94 mm
- net N$27: track 3.33 -> 2.67 mm
Other:
- board text added: "ESR NM8032 2020"
- board text removed: "ESR NM8032"

Commit message: .c
Parts:
- removed C19: 470x6v3, rcl:E15-5
- C14, C8: device HWProgUSB:RCL_E2,5-7 -> HWProgUSB:RCL_E2,5-5
- C18, C21: device HWProgUSB:RCL_E2-5 -> HWProgUSB:RCL_E2,5-5
- C9: value 470x6v3 -> 560x6v3; device rcl:E15-5 -> HWProgUSB:HWPROGUSB_RCL_E3,5-8
- moved C9 5.13 mm to (13.0, 42.9)
Connections:
- net GNDS: no longer C19.-
- net VCCS: no longer C19.+
Routing:
- net GNDS: track 25.4 -> 21.7 mm
- net GND: track 299.6 -> 297.9 mm
- net VCCS: track 20.9 -> 20.1 mm

Commit message: .
Parts:
- added R3': 10, rcl:M0805
- L3: device rcl:0204/5 -> rcl:0207/10
- R3: value 110 -> 100
- moved L3 5.40 mm to (10.2, 97.5), turned to 180 degrees
- moved R2 5.08 mm to (19.1, 43.5)
- moved R3 3.82 mm to (16.2, 41.0), turned to 90 degrees
- moved C8 1.59 mm to (6.35, 92.4)
- turned S2 to 180 degrees
Connections:
- new net N$17: R3'.2, R3.1
- net N$40: now also R3'.1; no longer R3.1
Routing:
- net N$26: track 24.6 -> 20.2 mm
- net VCC/2: track 38.0 -> 42.3 mm
- net N$38: track 26.3 -> 29.1 mm
- net N$17: track 0.00 -> 2.57 mm
- net GND: track 297.9 -> 296.5 mm
Other:
- board text added: "X1 X10"

Commit message: .
Parts:
- C5: device rcl:E2,5-5 -> rcl:E2-5
- moved R3 1.93 mm to (18.1, 41.3)
- moved C9 1.00 mm to (14.0, 43.2)
- moved VD2 1.00 mm to (8.89, 41.6)
- moved DD1 1.00 mm to (1.59, 42.5)
- moved C3 1.00 mm to (5.40, 48.9)
- moved VD1 1.00 mm to (8.89, 43.8)
- moved C2 1.00 mm to (7.62, 42.9)
- moved C1 0.71 mm to (1.91, 36.5)
- moved R1 0.63 mm to (-2.22, 36.2)
- moved R2 0.63 mm to (19.1, 44.1)
- moved C5 0.32 mm to (6.67, 51.4)
Routing:
- net N$26: track 20.2 -> 17.6 mm
- net GND: track 296.5 -> 294.8 mm
- net GNDS: track 21.7 -> 22.8 mm
- net N$17: track 2.57 -> 1.91 mm
