File: ESR_NM8032.brd (EAGLE design)
At the start: 34.9 x 90.8 mm, 80 parts, among them J1 0

Commit message: .
Parts:
- removed C22: 100n, rcl:C0805
- X1, X2: device pinhead:1X02 -> Разъёмы штырьковые 2.54мм:1X02
- moved C13 18.9 mm to (19.1, 85.4)
- moved C16 18.9 mm to (22.5, 84.8)
- moved C17 18.9 mm to (4.13, 72.7)
- moved C5 18.9 mm to (14.0, 34.0)
- moved C7 18.9 mm to (12.1, 64.5)
- moved DA4 18.9 mm to (18.7, 89.5)
- moved HL1 18.9 mm to (33.0, 87.6)
- moved HL10 18.9 mm to (33.0, 47.6)
- moved HL3 18.9 mm to (33.0, 78.7)
- moved HL5 18.9 mm to (33.0, 69.8)
- moved HL6 18.9 mm to (33.0, 65.4)
- moved HL8 18.9 mm to (33.0, 56.5)
- moved J1 18.9 mm to (21.6, 67.6)
- moved L2.2 18.9 mm to (17.8, 95.2)
- moved R14 18.9 mm to (16.8, 93.3)
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Connections:
- net GND: no longer C22.2
- net V+: no longer C22.1
Routing:
- net N$23: track 28.8 -> 35.7 mm
- net GNDS: track 22.8 -> 16.9 mm
- net GND: track 294.8 -> 297.5 mm
- net N$52: track 0.00 -> 1.91 mm
- net N$51: track 0.00 -> 1.91 mm
- net N$24: track 31.2 -> 31.7 mm
Other:
- board text added: "1/10 0.1 0.2 0.3 0.4 0.5 0.8 1.1 1.5 2.1 3"
- board text added: "R03"
- board text removed: "1/10 1/1 0.1 1.3 0.2 1.9 0.3 2.7 0.4 3.8 0.5 5.3 0.8 7.5 1.1 10.6 1.5 15 2.1 21.2 3 30"

Commit message: .
Parts:
- DA5: value 78l06 -> 78L06
- R15: value 2k4 -> 1k5(2k4 6v)
- R16: value 9k1 -> 7k5(9k1 6v)
Changed lines of the file:
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@@
 <layer number="35" name="tGlue" color="7" fill="4" visible="no" active="yes"/>
 <layer number="36" name="bGlue" color="7" fill="5" visible="no" active="yes"/>
-<layer number="37" name="tTest" color="7" fill="1" visible="no" active="yes"/>
-<layer number="38" name="bTest" color="7" fill="1" visible="no" active="yes"/>
+<layer number="37" name="tTest" color="7" fill="1" visible="yes" active="yes"/>
+<layer number="38" name="bTest" color="7" fill="1" visible="yes" active="yes"/>
 <layer number="39" name="tKeepout" color="4" fill="11" visible="no" active="yes"/>
 <layer number="40" name="bKeepout" color="1" fill="11" visible="no" active="yes"/>
@@
 <layer number="101" name="Patch_Top" color="12" fill="4" visible="yes" active="yes"/>
 <layer number="102" name="Vscore" color="7" fill="1" visible="yes" active="yes"/>
-<layer number="103" name="tMap" color="7" fill="1" visible="yes" active="yes"/>
-<layer number="104" name="Name" color="16" fill="1" visible="yes" active="yes"/>
+<layer number="103" name="tMap" color="7" fill="1" visible="no" active="yes"/>
+<layer number="104" name="Name" color="16" fill="1" visible="no" active="yes"/>
 <layer number="105" name="tPlate" color="7" fill="1" visible="yes" active="yes"/>
 <layer number="106" name="bPlate" color="7" fill="1" visible="yes" active="yes"/>
@@
 <layer number="114" name="bJumper" color="7" fill="1" visible="yes" active="yes"/>
 <layer number="115" name="GND" color="7" fill="1" visible="yes" active="yes"/>
-<layer number="116" name="Patch_BOT" color="9" fill="4" visible="yes" active="yes"/>
+<layer number="116" name="Patch_BOT" color="9" fill="4" visible="no" active="yes"/>
 <layer number="117" name="tJumper" color="9" fill="1" visible="yes" active="yes"/>
 <layer number="118" name="Rect_Pads" color="7" fill="1" visible="no" active="no"/>
+<layer number="119" name="119" color="7" fill="1" visible="yes" active="yes"/>
+<layer number="120" name="120" color="7" fill="1" visible="yes" active="yes"/>
 <layer number="121" name="_tsilk" color="7" fill="1" visible="yes" active="yes"/>
 <layer number="122" name="_bsilk" color="7" fill="1" visible="yes" active="yes"/>
@@
 <layer number="127" name="_tValues" color="7" fill="1" visible="yes" active="yes"/>
 <layer number="128" name="_bValues" color="7" fill="1" visible="yes" active="yes"/>
+<layer number="129" name="129" color="7" fill="1" visible="yes" active="yes"/>
+<layer number="130" name="130" color="7" fill="1" visible="no" active="yes"/>
 <layer number="131" name="tAdjust" color="7" fill="1" visible="yes" active="yes"/>
 <layer number="132" name="bAdjust" color="7" fill="1" visible="yes" active="yes"/>
+<layer number="133" name="133" color="7" fill="1" visible="no" active="yes"/>
 <layer number="144" name="Drill_legend" color="7" fill="1" visible="yes" active="yes"/>
 <layer number="150" name="Notes" color="7" fill="1" visible="yes" active="yes"/>
 <layer number="151" name="HeatSink" color="7" fill="1" visible="yes" active="yes"/>
-<layer number="152" name="_bDocu" color="7" fill="1" visible="yes" active="yes"/>
+<layer number="152" name="_bDocu" color="7" fill="1" visible="no" active="yes"/>
 <layer number="153" name="FabDoc1" color="7" fill="1" visible="yes" active="yes"/>
 <layer number="154" name="FabDoc2" color="7" fill="1" visible="yes" active="yes"/>
 <layer number="155" name="FabDoc3" color="7" fill="1" visible="yes" active="yes"/>
 <layer number="199" name="Contour" color="7" fill="1" visible="yes" active="yes"/>
-<layer number="200" name="200bmp" color="1" fill="10" visible="yes" active="yes"/>
-<layer number="201" name="201bmp" color="2" fill="10" visible="yes" active="yes"/>
-<layer number="202" name="202bmp" color="3" fill="10" visible="yes" active="yes"/>
-<layer number="203" name="203bmp" color="4" fill="10" visible="yes" active="yes"/>
-<layer number="204" name="204bmp" color="5" fill="10" visible="yes" active="yes"/>
-<layer number="205" name="205bmp" color="6" fill="10" visible="yes" active="yes"/>
-<layer number="206" name="206bmp" color="7" fill="10" visible="yes" active="yes"/>
-<layer number="207" name="207bmp" color="8" fill="10" visible="yes" active="yes"/>
-<layer number="208" name="208bmp" color="9" fill="10" visible="yes" active="yes"/>
+<layer number="200" name="200bmp" color="1" fill="10" visible="no" active="yes"/>
+<layer number="201" name="201bmp" color="2" fill="10" visible="no" active="yes"/>
+<layer number="202" name="202bmp" color="3" fill="10" visible="no" active="yes"/>
+<layer number="203" name="203bmp" color="4" fill="10" visible="no" active="yes"/>
+<layer number="204" name="204bmp" color="5" fill="10" visible="no" active="yes"/>
+<layer number="205" name="205bmp" color="6" fill="10" visible="no" active="yes"/>
+<layer number="206" name="206bmp" color="7" fill="10" visible="no" active="yes"/>
+<layer number="207" name="207bmp" color="8" fill="10" visible="no" active="yes"/>
+<layer number="208" name="208bmp" color="9" fill="10" visible="no" active="yes"/>
 <layer number="209" name="209bmp" color="7" fill="1" visible="yes" active="yes"/>
 <layer number="210" name="210bmp" color="7" fill="1" visible="yes" active="yes"/>
@@
 <attribute name="VALUE" x="20.32" y="87.63" size="1.27" layer="28" rot="MR90"/>
 </element>
-<element name="R16" library="rcl" package="M0805" value="9k1" x="22.225" y="96.8375" smashed="yes" rot="MR180">
+<element name="R16" library="rcl" package="M0805" value="7k5(9k1 6v)" x="22.225" y="96.8375" smashed="yes" rot="MR180">
 <attribute name="NAME" x="23.495" y="94.2975" size="1.27" layer="26" rot="MR0"/>
 <attribute name="VALUE" x="22.5425" y="93.6625" size="1.27" layer="28" rot="MR180"/>
 </element>
-<element name="R15" library="rcl" package="M0805" value="2k4" x="13.0175" y="96.8375" smashed="yes" rot="MR180">
+<element name="R15" library="rcl" package="M0805" value="1k5(2k4 6v)" x="13.0175" y="96.8375" smashed="yes" rot="MR180">
 <attribute name="NAME" x="11.1125" y="96.2025" size="1.27" layer="26" rot="MR0"/>
 <attribute name="VALUE" x="9.8425" y="90.805" size="1.27" layer="28" rot="MR90"/>
@@
 <attribute name="VALUE" x="10.795" y="50.546" size="1.27" layer="27" ratio="10"/>
 </element>
-<element name="DA5" library="ct-pack" package="SOT89R" value="78l06" x="7.62" y="72.0725" smashed="yes" rot="MR90">
+<element name="DA5" library="ct-pack" package="SOT89R" value="78L06" x="7.62" y="72.0725" smashed="yes" rot="MR90">
 <attribute name="NAME" x="10.1425" y="76.75" size="1.27" layer="26" rot="MR0"/>
 <attribute name="VALUE" x="10.7775" y="74.915" size="1.27" layer="28" rot="MR0"/>

Commit message: .
Parts:
- moved C8 0.32 mm to (13.7, 75.2)
Changed lines of the file:
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@@
 <attribute name="VALUE" x="1.905" y="76.2" size="1.27" layer="28" rot="MR180"/>
 </element>
-<element name="C8" library="HWProgUSB" package="RCL_E2,5-5" value="100µ 16V" x="13.6525" y="74.93" smashed="yes" rot="R270">
-<attribute name="NAME" x="10.668" y="77.597" size="1.27" layer="25" ratio="10"/>
-<attribute name="VALUE" x="15.113" y="77.1525" size="1.27" layer="27" ratio="10"/>
+<element name="C8" library="HWProgUSB" package="RCL_E2,5-5" value="100µ 16V" x="13.6525" y="75.2475" smashed="yes" rot="R270">
+<attribute name="NAME" x="10.668" y="77.9145" size="1.27" layer="25" ratio="10"/>
+<attribute name="VALUE" x="15.113" y="77.47" size="1.27" layer="27" ratio="10"/>
 </element>
 <element name="U$1" library="ESR_NM8032" package="LR03" value="" x="5.715" y="30.1625" rot="R90"/>
@@
 <wire x1="8.52" y1="72.0725" x2="10.4775" y2="72.0725" width="1.27" layer="16"/>
 <wire x1="13.401" y1="70.4825" x2="13.6525" y2="70.485" width="1.016" layer="16"/>
-<wire x1="13.6525" y1="70.485" x2="13.6525" y2="73.66" width="1.016" layer="16"/>
-<wire x1="13.6525" y1="73.9775" x2="13.6525" y2="73.66" width="1.016" layer="16"/>
+<wire x1="13.6525" y1="70.485" x2="13.6525" y2="73.9775" width="1.016" layer="16"/>
 <wire x1="17.78" y1="70.8025" x2="15.5575" y2="70.8025" width="1.016" layer="16"/>
 <wire x1="15.5575" y1="70.8025" x2="14.224" y2="70.8025" width="1.016" layer="16"/>
@@
 <wire x1="4.2125" y1="73.5725" x2="4.1275" y2="73.6575" width="0.6096" layer="16"/>
 <contactref element="R17" pad="1"/>
-<wire x1="13.6525" y1="76.2" x2="11.1125" y2="76.2" width="1.27" layer="16"/>
-<wire x1="11.1125" y1="76.2" x2="10.16" y2="75.2475" width="1.27" layer="16"/>
+<wire x1="13.6525" y1="76.5175" x2="11.43" y2="76.5175" width="1.27" layer="16"/>
+<wire x1="11.43" y1="76.5175" x2="10.16" y2="75.2475" width="1.27" layer="16"/>
 <wire x1="10.16" y1="75.2475" x2="6.6675" y2="75.2475" width="1.27" layer="16"/>
 <wire x1="28.2575" y1="86.995" x2="28.2575" y2="82.55" width="0.6096" layer="16"/>
@@
 <wire x1="28.2575" y1="86.995" x2="31.4325" y2="90.17" width="0.6096" layer="16"/>
 <wire x1="31.4325" y1="90.17" x2="32.07" y2="90.17" width="0.6096" layer="16"/>
-<wire x1="13.6525" y1="76.2" x2="13.6525" y2="78.74" width="0.6096" layer="16"/>
+<wire x1="13.6525" y1="76.5175" x2="13.6525" y2="78.74" width="0.6096" layer="16"/>
 <wire x1="13.6525" y1="78.74" x2="12.3825" y2="80.01" width="0.6096" layer="16"/>
-<wire x1="23.921446875" y1="78.213946875" x2="15.666446875" y2="78.213946875" width="0.6096" layer="16"/>
-<wire x1="15.666446875" y1="78.213946875" x2="13.6525" y2="76.2" width="0.6096" layer="16"/>
+<wire x1="23.921446875" y1="78.213946875" x2="15.348946875" y2="78.213946875" width="0.6096" layer="16"/>
+<wire x1="15.348946875" y1="78.213946875" x2="13.6525" y2="76.5175" width="0.6096" layer="16"/>
 </signal>
 <signal name="+6V">

Commit message: .2
Parts:
- added JB: (no value), jumper:SJ
- added R28*: 2k7, rcl:R0805
- moved R17 47.0 mm to (33.3, 43.2)
Connections:
- removed net VCC/2: C17.1, C8.+, DA5.1, L3.2, R17.1
- new net N$54: DA3.9, JB.2
- new net N$55: C17.1, C8.+, DA5.1, L3.2
- net N$28: now also R28*.2
- net N$3: now also R28*.1
- net N$41: now also JB.1, R17.1; no longer DA3.9
Routing:
- net VCC/2: track 42.0 -> 0.00 mm
- net N$55: track 0.00 -> 15.3 mm
- net N$41: track 60.3 -> 66.0 mm
- net N$28: track 42.7 -> 47.0 mm
- net N$3: track 19.5 -> 22.3 mm
- net N$54: track 0.00 -> 2.73 mm

Commit message: .
Parts:
- DA2: value K157DA1 -> К157ДА1
- DD1: value 4049D -> HEF4049BT
Changed lines of the file:
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@@
 <attribute name="VALUE" x="18.7325" y="74.93" size="1.27" layer="27" ratio="10"/>
 </element>
-<element name="DD1" library="40xx" package="SO16" value="4049D" x="8.89" y="25.0825" rot="MR270"/>
+<element name="DD1" library="40xx" package="SO16" value="HEF4049BT" x="8.89" y="25.0825" rot="MR270"/>
 <element name="C1" library="rcl" package="C0805" value="330" x="9.2075" y="19.05" smashed="yes" rot="MR180">
 <attribute name="NAME" x="10.16" y="16.8275" size="1.27" layer="26" rot="MR0"/>
@@
 <attribute name="VALUE" x="16.598896875" y="79.6036" size="0.9906" layer="27" ratio="10"/>
 </element>
-<element name="DA2" library="ESR_NM8032" package="DIL14" value="K157DA1" x="21.59" y="43.4975" smashed="yes">
+<element name="DA2" library="ESR_NM8032" package="DIL14" value="К157ДА1" x="21.59" y="43.4975" smashed="yes">
 <attribute name="NAME" x="18.542" y="49.276" size="1.27" layer="25" ratio="10"/>
 <attribute name="VALUE" x="23.114" y="49.2125" size="1.27" layer="27" ratio="10"/>

Commit message: .
Parts:
- R6: value 10k -> 56k
Changed lines of the file:
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@@
 <attribute name="VALUE" x="30.099" y="34.7345" size="1.27" layer="27" ratio="10"/>
 </element>
-<element name="R6" library="rcl" package="R0805" value="10k" x="25.0825" y="36.195" smashed="yes" rot="MR180">
+<element name="R6" library="rcl" package="R0805" value="56k" x="25.0825" y="36.195" smashed="yes" rot="MR180">
 <attribute name="NAME" x="25.0825" y="34.925" size="1.27" layer="26" rot="MR180"/>
 <attribute name="VALUE" x="24.4475" y="38.735" size="1.27" layer="28" rot="MR180"/>

Commit message: .
Parts:
- R13: value 0.5-1 -> 0.5
Changed lines of the file:
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@@
 <wire x1="35.54" y1="98.4125" x2="0.635" y2="98.4125" width="0" layer="20"/>
 <wire x1="0.635" y1="98.4125" x2="0.635" y2="7.62" width="0" layer="20"/>
-<dimension x1="36.195" y1="98.425" x2="36.195" y2="7.62" x3="38.735" y3="53.0225" textsize="1.778" layer="21" dtype="vertical"/>
+<dimension x1="36.195" y1="98.425" x2="36.195" y2="7.62" x3="41.5925" y3="53.0225" textsize="1.778" layer="21" dtype="vertical"/>
 <text x="0.9525" y="14.2875" size="1.778" layer="51">1/1
 1.3
@@
 <text x="3.81" y="80.3275" size="1.778" layer="21" font="vector" ratio="15">R03</text>
 <circle x="13.97" y="93.0275" radius="1.419903125" width="0.1524" layer="21"/>
+<rectangle x1="0.635" y1="14.605" x2="2.54" y2="72.39" layer="30"/>
+<rectangle x1="0.635" y1="72.39" x2="2.2225" y2="97.79" layer="30"/>
+<dimension x1="36.195" y1="87.63" x2="36.195" y2="83.185" x3="38.4175" y3="85.4075" textsize="1.778" layer="21" dtype="vertical"/>
 </plain>
 <attributes>
@@
 <attribute name="VALUE" x="22.5425" y="93.98" size="1.27" layer="28" rot="MR0"/>
 </element>
-<element name="R13" library="rcl" package="M1206" value="0.5-1" x="13.335" y="89.8525" smashed="yes" rot="MR90">
+<element name="R13" library="rcl" package="M1206" value="0.5" x="13.335" y="89.8525" smashed="yes" rot="MR90">
 <attribute name="NAME" x="10.795" y="88.265" size="1.27" layer="26" rot="MR90"/>
 <attribute name="VALUE" x="20.32" y="87.63" size="1.27" layer="28" rot="MR90"/>
@@
 <wire x1="16.51" y1="45.7225" x2="16.51" y2="47.3075" width="0.6096" layer="16"/>
 <wire x1="19.3675" y1="88.265" x2="20.0025" y2="87.63" width="0.6096" layer="16"/>
-<wire x1="1.5875" y1="15.24" x2="1.5875" y2="71.755" width="1.4224" layer="16"/>
+<wire x1="1.5875" y1="15.24" x2="1.5875" y2="71.755" width="1.778" layer="16"/>
 <wire x1="1.5875" y1="71.755" x2="1.5875" y2="83.185" width="1.4224" layer="16"/>
 <wire x1="1.5875" y1="83.185" x2="1.5875" y2="97.4725" width="1.4224" layer="16"/>
